File: adc.kicad_sch (KiCad schematic)
At the start: 18 parts, among them U701 ADS8665IPWR

Commit message: add i-transduce schematic
Other:
- title: Power Supply Sink -> Measurement
Changed lines of the file:
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@@
 	(paper "A4")
 	(title_block
-		(title "Power Supply Sink")
-		(date "2024-12-14")
-		(rev "1.0.0")
+		(title "Measurement")
+		(date "2025-02-22")
+		(rev "0.0.0")
 		(company "Open Battery Tester")
 		(comment 1 "Analog Digital Converter")
