File: adc.kicad_sch (KiCad schematic)
At the start: 18 parts, among them U701 ADS8665IPWR

Commit message: add export of symbol libray, edit symbol links
Parts:
- C701, C702, C703, C704, C705, C706, C707: symbol pss:C -> meas:C
- D701: symbol pss:LED -> meas:LED
- JP701: symbol pss:SolderJumper_2_Open -> meas:SolderJumper_2_Open
- JP702: symbol pss:SolderJumper_2_Bridged -> meas:SolderJumper_2_Bridged
- R701, R702, R703, R704: symbol pss:R -> meas:R
- TP701, TP702, TP703: symbol pss:TestPoint -> meas:TestPoint
- U701: symbol pss:ADS866x -> meas:ADS866x
Changed lines of the file:
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@@
 	)
 	(symbol
-		(lib_id "pss:C")
+		(lib_id "meas:C")
 		(at 88.9 91.44 180)
 		(unit 1)
@@
 	)
 	(symbol
-		(lib_id "pss:R")
+		(lib_id "meas:R")
 		(at 177.8 85.09 90)
 		(unit 1)
@@
 	)
 	(symbol
-		(lib_id "pss:C")
+		(lib_id "meas:C")
 		(at 168.91 102.87 180)
 		(unit 1)
@@
 	)
 	(symbol
-		(lib_id "pss:R")
+		(lib_id "meas:R")
 		(at 88.9 120.65 0)
 		(unit 1)
@@
 	)
 	(symbol
-		(lib_id "pss:TestPoint")
+		(lib_id "meas:TestPoint")
 		(at 171.45 99.06 270)
 		(unit 1)
@@
 	)
 	(symbol
-		(lib_id "pss:ADS866x")
+		(lib_id "meas:ADS866x")
 		(at 137.16 91.44 0)
 		(unit 1)
@@
 	)
 	(symbol
-		(lib_id "pss:C")
+		(lib_id "meas:C")
 		(at 168.91 88.9 180)
 		(unit 1)
@@
 	)
 	(symbol
-		(lib_id "pss:R")
+		(lib_id "meas:R")
 		(at 177.8 92.71 90)
 		(unit 1)
@@
 	)
 	(symbol
-		(lib_id "pss:TestPoint")
+		(lib_id "meas:TestPoint")
 		(at 184.15 85.09 0)
 		(unit 1)
@@
 	)
 	(symbol
-		(lib_id "pss:TestPoint")
+		(lib_id "meas:TestPoint")
 		(at 88.9 104.14 0)
 		(unit 1)
@@
 	)
 	(symbol
-		(lib_id "pss:C")
+		(lib_id "meas:C")
 		(at 140.97 67.31 180)
 		(unit 1)
@@
 	)
 	(symbol
-		(lib_id "pss:R")
+		(lib_id "meas:R")
 		(at 82.55 86.36 90)
 		(unit 1)
@@
 	)
 	(symbol
-		(lib_id "pss:SolderJumper_2_Open")
+		(lib_id "meas:SolderJumper_2_Open")
 		(at 88.9 81.28 270)
 		(unit 1)
@@
 	)
 	(symbol
-		(lib_id "pss:C")
+		(lib_id "meas:C")
 		(at 219.71 102.87 180)
 		(unit 1)
@@
 	)
 	(symbol
-		(lib_id "pss:C")
+		(lib_id "meas:C")
 		(at 125.73 67.31 180)
 		(unit 1)
@@
 	)
 	(symbol
-		(lib_id "pss:C")
+		(lib_id "meas:C")
 		(at 203.2 102.87 180)
 		(unit 1)
@@
 	)
 	(symbol
-		(lib_id "pss:LED")
+		(lib_id "meas:LED")
 		(at 88.9 130.81 90)
 		(unit 1)
@@
 	)
 	(symbol
-		(lib_id "pss:SolderJumper_2_Bridged")
+		(lib_id "meas:SolderJumper_2_Bridged")
 		(at 88.9 109.22 90)
 		(unit 1)

Commit message: add export of footprint library, edit footprint links
Parts:
- C701, C702, C703, C706: footprint pss:C_0603_1608Metric_Pad1.08x0.95mm_HandSolder -> meas:C_0603_1608Metric_Pad1.08x0.95mm_HandSolder
- C704: footprint pss:C_1206_3216Metric_Pad1.33x1.80mm_HandSolder -> meas:C_1206_3216Metric_Pad1.33x1.80mm_HandSolder
- C705, C707: footprint pss:C_1210_3225Metric_Pad1.33x2.70mm_HandSolder -> meas:C_1210_3225Metric_Pad1.33x2.70mm_HandSolder
- D701: footprint pss:LED_0805_2012Metric_Pad1.15x1.40mm_HandSolder -> meas:LED_0805_2012Metric_Pad1.15x1.40mm_HandSolder
- JP701: footprint pss:SolderJumper-2_P1.3mm_Open_RoundedPad1.0x1.5mm -> meas:SolderJumper-2_P1.3mm_Open_RoundedPad1.0x1.5mm
- JP702: footprint pss:SolderJumper-2_P1.3mm_Bridged-Soldermask-Paste_RoundedPad1.0x1.5mm -> meas:SolderJumper-2_P1.3mm_Bridged-Soldermask-Paste_RoundedPad1.0x1.5mm
- R701, R702, R703, R704: footprint pss:R_1210_3225Metric_Pad1.30x2.65mm_HandSolder -> meas:R_1210_3225Metric_Pad1.30x2.65mm_HandSolder
- TP701, TP702, TP703: footprint pss:TP_0805_2012Metric -> meas:TP_0805_2012Metric
- U701: footprint pss:TSSOP-16_4.4x5mm_P0.65mm -> meas:TSSOP-16_4.4x5mm_P0.65mm
Changed lines of the file:
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@@
 			)
 		)
-		(property "Footprint" "pss:C_0603_1608Metric_Pad1.08x0.95mm_HandSolder"
+		(property "Footprint" "meas:C_0603_1608Metric_Pad1.08x0.95mm_HandSolder"
 			(at 87.9348 87.63 0)
 			(effects
@@
 			)
 		)
-		(property "Footprint" "pss:R_1210_3225Metric_Pad1.30x2.65mm_HandSolder"
+		(property "Footprint" "meas:R_1210_3225Metric_Pad1.30x2.65mm_HandSolder"
 			(at 177.8 86.868 90)
 			(effects
@@
 			)
 		)
-		(property "Footprint" "pss:C_1210_3225Metric_Pad1.33x2.70mm_HandSolder"
+		(property "Footprint" "meas:C_1210_3225Metric_Pad1.33x2.70mm_HandSolder"
 			(at 167.9448 99.06 0)
 			(effects
@@
 			)
 		)
-		(property "Footprint" "pss:R_1210_3225Metric_Pad1.30x2.65mm_HandSolder"
+		(property "Footprint" "meas:R_1210_3225Metric_Pad1.30x2.65mm_HandSolder"
 			(at 87.122 120.65 90)
 			(effects
@@
 			)
 		)
-		(property "Footprint" "pss:TP_0805_2012Metric"
+		(property "Footprint" "meas:TP_0805_2012Metric"
 			(at 171.45 104.14 0)
 			(effects
@@
 			)
 		)
-		(property "Footprint" "pss:TSSOP-16_4.4x5mm_P0.65mm"
+		(property "Footprint" "meas:TSSOP-16_4.4x5mm_P0.65mm"
 			(at 137.16 133.35 0)
 			(effects
@@
 			)
 		)
-		(property "Footprint" "pss:C_1206_3216Metric_Pad1.33x1.80mm_HandSolder"
+		(property "Footprint" "meas:C_1206_3216Metric_Pad1.33x1.80mm_HandSolder"
 			(at 167.9448 85.09 0)
 			(effects
@@
 			)
 		)
-		(property "Footprint" "pss:R_1210_3225Metric_Pad1.30x2.65mm_HandSolder"
+		(property "Footprint" "meas:R_1210_3225Metric_Pad1.30x2.65mm_HandSolder"
 			(at 177.8 94.488 90)
 			(effects
@@
 			)
 		)
-		(property "Footprint" "pss:TP_0805_2012Metric"
+		(property "Footprint" "meas:TP_0805_2012Metric"
 			(at 189.23 85.09 0)
 			(effects
@@
 			)
 		)
-		(property "Footprint" "pss:TP_0805_2012Metric"
+		(property "Footprint" "meas:TP_0805_2012Metric"
 			(at 93.98 104.14 0)
 			(effects
@@
 			)
 		)
-		(property "Footprint" "pss:C_0603_1608Metric_Pad1.08x0.95mm_HandSolder"
+		(property "Footprint" "meas:C_0603_1608Metric_Pad1.08x0.95mm_HandSolder"
 			(at 140.0048 63.5 0)
 			(effects
@@
 			)
 		)
-		(property "Footprint" "pss:R_1210_3225Metric_Pad1.30x2.65mm_HandSolder"
+		(property "Footprint" "meas:R_1210_3225Metric_Pad1.30x2.65mm_HandSolder"
 			(at 82.55 88.138 90)
 			(effects
@@
 			)
 		)
-		(property "Footprint" "pss:SolderJumper-2_P1.3mm_Open_RoundedPad1.0x1.5mm"
+		(property "Footprint" "meas:SolderJumper-2_P1.3mm_Open_RoundedPad1.0x1.5mm"
 			(at 88.9 81.28 0)
 			(effects
@@
 			)
 		)
-		(property "Footprint" "pss:C_1210_3225Metric_Pad1.33x2.70mm_HandSolder"
+		(property "Footprint" "meas:C_1210_3225Metric_Pad1.33x2.70mm_HandSolder"
 			(at 218.7448 99.06 0)
 			(effects
@@
 			)
 		)
-		(property "Footprint" "pss:C_0603_1608Metric_Pad1.08x0.95mm_HandSolder"
+		(property "Footprint" "meas:C_0603_1608Metric_Pad1.08x0.95mm_HandSolder"
 			(at 124.7648 63.5 0)
 			(effects
@@
 			)
 		)
-		(property "Footprint" "pss:C_0603_1608Metric_Pad1.08x0.95mm_HandSolder"
+		(property "Footprint" "meas:C_0603_1608Metric_Pad1.08x0.95mm_HandSolder"
 			(at 202.2348 99.06 0)
 			(effects
@@
 			)
 		)
-		(property "Footprint" "pss:LED_0805_2012Metric_Pad1.15x1.40mm_HandSolder"
+		(property "Footprint" "meas:LED_0805_2012Metric_Pad1.15x1.40mm_HandSolder"
 			(at 88.9 130.81 0)
 			(effects
@@
 			)
 		)
-		(property "Footprint" "pss:SolderJumper-2_P1.3mm_Bridged-Soldermask-Paste_RoundedPad1.0x1.5mm"
+		(property "Footprint" "meas:SolderJumper-2_P1.3mm_Bridged-Soldermask-Paste_RoundedPad1.0x1.5mm"
 			(at 88.9 109.22 0)
 			(effects
