File: digital-interface.kicad_sch (KiCad schematic)
At the start: 37 parts, among them U301 Si8641BD-B-IS2, U302 R05C05TE05S

Commit message: add i-transduce schematic
Other:
- title: Power Supply Sink -> Measurement
Changed lines of the file:
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@@
 	(paper "A4")
 	(title_block
-		(title "Power Supply Sink")
+		(title "Measurement")
 		(date "2025-02-22")
-		(rev "1.1.2")
+		(rev "0.0.0")
 		(company "Open Battery Tester")
 		(comment 1 "Digital Interface")
