File: meas.kicad_sch (KiCad schematic)
At the start: 13 parts, among them J101 Conn_01x06_Socket, J102 Conn_01x02_Socket, J103 Conn_01x02_Socket, J104 Conn_01x02_Socket, J105 Conn_01x02_Socket

Commit message: add export of symbol libray, edit symbol links
Parts:
- D101, D102: symbol enclosure:D_TVS -> meas:D_TVS
- F101: symbol enclosure:Fuse_Socket_1 -> meas:Fuse_Socket_1
- F102: symbol enclosure:Fuse -> meas:Fuse
- J101: symbol pss:Conn_01x06_Socket -> meas:Conn_01x06_Socket
- J102, J103, J104, J105: symbol pss:Conn_01x02_Socket -> meas:Conn_01x02_Socket
- R101, R102, R103, R104: symbol pss:R -> meas:R
Changed lines of the file:
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@@
 	)
 	(symbol
-		(lib_id "pss:R")
+		(lib_id "meas:R")
 		(at 222.25 43.18 270)
 		(unit 1)
@@
 	)
 	(symbol
-		(lib_id "pss:Conn_01x02_Socket")
+		(lib_id "meas:Conn_01x02_Socket")
 		(at 261.62 81.28 0)
 		(unit 1)
@@
 	)
 	(symbol
-		(lib_id "enclosure:GND")
+		(lib_id "meas:GND")
 		(at 50.8 80.01 90)
 		(unit 1)
@@
 	)
 	(symbol
-		(lib_id "power:+5VA")
+		(lib_id "meas:+5VA")
 		(at 118.11 33.02 0)
 		(unit 1)
@@
 	)
 	(symbol
-		(lib_id "pss:Conn_01x06_Socket")
+		(lib_id "meas:Conn_01x06_Socket")
 		(at 38.1 43.18 0)
 		(mirror y)
@@
 	)
 	(symbol
-		(lib_id "pss:R")
+		(lib_id "meas:R")
 		(at 215.9 127 0)
 		(unit 1)
@@
 	)
 	(symbol
-		(lib_id "enclosure:GND")
+		(lib_id "meas:GND")
 		(at 120.65 146.05 0)
 		(unit 1)
@@
 	)
 	(symbol
-		(lib_id "enclosure:D_TVS")
+		(lib_id "meas:D_TVS")
 		(at 241.3 50.8 90)
 		(unit 1)
@@
 	)
 	(symbol
-		(lib_id "pss:R")
+		(lib_id "meas:R")
 		(at 215.9 50.8 180)
 		(unit 1)
@@
 	(symbol
 		(lib_name "Fuse_Socket_1")
-		(lib_id "enclosure:Fuse_Socket_1")
+		(lib_id "meas:Fuse_Socket_1")
 		(at 248.92 83.82 270)
 		(unit 1)
@@
 	)
 	(symbol
-		(lib_id "enclosure:D_TVS")
+		(lib_id "meas:D_TVS")
 		(at 241.3 127 90)
 		(unit 1)
@@
 	)
 	(symbol
-		(lib_id "pss:Conn_01x02_Socket")
+		(lib_id "meas:Conn_01x02_Socket")
 		(at 38.1 80.01 0)
 		(mirror y)
@@
 	)
 	(symbol
-		(lib_id "pss:Conn_01x02_Socket")
+		(lib_id "meas:Conn_01x02_Socket")
 		(at 259.08 116.84 0)
 		(unit 1)
@@
 	)
 	(symbol
-		(lib_id "enclosure:Fuse")
+		(lib_id "meas:Fuse")
 		(at 248.92 83.82 90)
 		(unit 1)
@@
 	)
 	(symbol
-		(lib_id "pss:R")
+		(lib_id "meas:R")
 		(at 222.25 119.38 90)
 		(unit 1)
@@
 	)
 	(symbol
-		(lib_id "pss:Conn_01x02_Socket")
+		(lib_id "meas:Conn_01x02_Socket")
 		(at 259.08 40.64 0)
 		(unit 1)

Commit message: add export of footprint library, edit footprint links
Parts:
- D101, D102: footprint enclosure:D_SOD-323_HandSoldering -> meas:D_SOD-323_HandSoldering
- F101: footprint enclosure:FuseHolder_Blade_ATO_Littelfuse_FLR_178.6165 -> meas:FuseHolder_Blade_ATO_Littelfuse_FLR_178.6165
- J101: footprint pss:PhoenixContact_TDPT_2,5_6-SP-5,08_1x06_P5.08mm_Horizontal -> meas:PhoenixContact_TDPT_2,5_6-SP-5,08_1x06_P5.08mm_Horizontal
- J102, J103, J104, J105: footprint pss:PhoenixContact_TDPT_2,5_2-SP-5,08_1x02_P5.08mm_Horizontal -> meas:PhoenixContact_TDPT_2,5_2-SP-5,08_1x02_P5.08mm_Horizontal
- R101, R102, R103, R104: footprint pss:R_1210_3225Metric_Pad1.30x2.65mm_HandSolder -> meas:R_1210_3225Metric_Pad1.30x2.65mm_HandSolder
Changed lines of the file:
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@@
 			)
 		)
-		(property "Footprint" "pss:R_1210_3225Metric_Pad1.30x2.65mm_HandSolder"
+		(property "Footprint" "meas:R_1210_3225Metric_Pad1.30x2.65mm_HandSolder"
 			(at 222.25 41.402 90)
 			(effects
@@
 			)
 		)
-		(property "Footprint" "pss:PhoenixContact_TDPT_2,5_2-SP-5,08_1x02_P5.08mm_Horizontal"
+		(property "Footprint" "meas:PhoenixContact_TDPT_2,5_2-SP-5,08_1x02_P5.08mm_Horizontal"
 			(at 261.62 81.28 0)
 			(effects
@@
 			)
 		)
-		(property "Footprint" "pss:PhoenixContact_TDPT_2,5_6-SP-5,08_1x06_P5.08mm_Horizontal"
+		(property "Footprint" "meas:PhoenixContact_TDPT_2,5_6-SP-5,08_1x06_P5.08mm_Horizontal"
 			(at 38.1 43.18 0)
 			(effects
@@
 			)
 		)
-		(property "Footprint" "pss:R_1210_3225Metric_Pad1.30x2.65mm_HandSolder"
+		(property "Footprint" "meas:R_1210_3225Metric_Pad1.30x2.65mm_HandSolder"
 			(at 214.122 127 90)
 			(effects
@@
 			)
 		)
-		(property "Footprint" "enclosure:D_SOD-323_HandSoldering"
+		(property "Footprint" "meas:D_SOD-323_HandSoldering"
 			(at 241.3 50.8 0)
 			(effects
@@
 			)
 		)
-		(property "Footprint" "pss:R_1210_3225Metric_Pad1.30x2.65mm_HandSolder"
+		(property "Footprint" "meas:R_1210_3225Metric_Pad1.30x2.65mm_HandSolder"
 			(at 217.678 50.8 90)
 			(effects
@@
 			)
 		)
-		(property "Footprint" "enclosure:FuseHolder_Blade_ATO_Littelfuse_FLR_178.6165"
+		(property "Footprint" "meas:FuseHolder_Blade_ATO_Littelfuse_FLR_178.6165"
 			(at 248.92 82.042 90)
 			(effects
@@
 			)
 		)
-		(property "Footprint" "enclosure:D_SOD-323_HandSoldering"
+		(property "Footprint" "meas:D_SOD-323_HandSoldering"
 			(at 241.3 127 0)
 			(effects
@@
 			)
 		)
-		(property "Footprint" "pss:PhoenixContact_TDPT_2,5_2-SP-5,08_1x02_P5.08mm_Horizontal"
+		(property "Footprint" "meas:PhoenixContact_TDPT_2,5_2-SP-5,08_1x02_P5.08mm_Horizontal"
 			(at 38.1 80.01 0)
 			(effects
@@
 			)
 		)
-		(property "Footprint" "pss:PhoenixContact_TDPT_2,5_2-SP-5,08_1x02_P5.08mm_Horizontal"
+		(property "Footprint" "meas:PhoenixContact_TDPT_2,5_2-SP-5,08_1x02_P5.08mm_Horizontal"
 			(at 259.08 116.84 0)
 			(effects
@@
 			)
 		)
-		(property "Footprint" "pss:R_1210_3225Metric_Pad1.30x2.65mm_HandSolder"
+		(property "Footprint" "meas:R_1210_3225Metric_Pad1.30x2.65mm_HandSolder"
 			(at 222.25 121.158 90)
 			(effects
@@
 			)
 		)
-		(property "Footprint" "pss:PhoenixContact_TDPT_2,5_2-SP-5,08_1x02_P5.08mm_Horizontal"
+		(property "Footprint" "meas:PhoenixContact_TDPT_2,5_2-SP-5,08_1x02_P5.08mm_Horizontal"
 			(at 259.08 40.64 0)
 			(effects
