File: power.kicad_sch (KiCad schematic)
At the start: 14 parts, among them Q1001 DPLS350E, U1001 MC7805

Commit message: fix wrong fuse in bom
Parts:
- F1001: MPN 0287030.PXCN -> 0287001.PXCN; VPN 576-0287030.PXCN -> 576-0287001.PXCN
Changed lines of the file:
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@@
 			)
 		)
-		(property "MPN" "0287030.PXCN"
+		(property "MPN" "0287001.PXCN"
 			(at 81.28 93.98 0)
 			(effects
@@
 			)
 		)
-		(property "VPN" "576-0287030.PXCN"
+		(property "VPN" "576-0287001.PXCN"
 			(at 81.28 93.98 0)
 			(effects
